Commit message: Localisation con telemetria y kalman, gazebo con arucos pista

File: reto_final/urdf/puzzlebot_jetson_lidar_ed_v1.xacro (robot description, xacro)
@@ -262,4 +262,9 @@
         <origin xyz="${chassis_pos_x} ${chassis_pos_y} ${chassis_pos_z}" rpy="${chassis_pos_r} ${chassis_pos_p} ${chassis_pos_w}"/>
     </joint>
+    <joint name="world_to_base_footprint" type="fixed">
+        <parent link="world"/>
+        <child link="base_link"/>
+        <origin xyz="0 0 0" rpy="0 0 0"/>
+    </joint>
     <joint name="motor_left_joint" type="fixed">
         <parent link="base_link"/>
