Commit message: Bug 0 arreglado

File: reto_final/urdf/puzzlebot_jetson_lidar_ed_v1.gazebo.xacro (robot description, xacro)
@@ -208,5 +208,5 @@
         <plugin name="p3d_controller_ground_truth" filename="libgazebo_ros_p3d.so">
             <alwaysOn>$(arg ground_truth)</alwaysOn>
-            <frameName>world</frameName>
+            <frameName>odom</frameName>
             <bodyName>base_link</bodyName>
             <topicName>base_pose_ground_truth</topicName>

File: reto_final/urdf/puzzlebot_jetson_lidar_ed_v1.xacro (robot description, xacro)
@@ -236,7 +236,7 @@
         </inertial>
     </link>
-    <link name="laser">
-        <visual>
-            <origin xyz="${lidar_mesh_pos_x} ${lidar_mesh_pos_y} ${lidar_mesh_pos_z}" rpy="${lidar_mesh_pos_r} ${lidar_mesh_pos_p} ${lidar_mesh_pos_w}"/>
+    <link name="laser_link">
+        <visual>
+            <origin xyz="${lidar_mesh_pos_x} ${lidar_mesh_pos_y} ${lidar_mesh_pos_z}" rpy="${lidar_mesh_pos_r} ${lidar_mesh_pos_p} 0"/>
             <geometry>
                 <mesh filename="file://${mesh_puzzlebot_lidar_sensor}"/>
@@ -262,9 +262,4 @@
         <origin xyz="${chassis_pos_x} ${chassis_pos_y} ${chassis_pos_z}" rpy="${chassis_pos_r} ${chassis_pos_p} ${chassis_pos_w}"/>
     </joint>
-    <joint name="world_to_base_footprint" type="fixed">
-        <parent link="world"/>
-        <child link="base_link"/>
-        <origin xyz="0 0 0" rpy="0 0 0"/>
-    </joint>
     <joint name="motor_left_joint" type="fixed">
         <parent link="base_link"/>
@@ -305,5 +300,5 @@
         <parent link="lidar_base_link"/>
         <child link="laser"/>
-        <origin xyz="${lidar_pos_x} ${lidar_pos_y} ${lidar_pos_z}" rpy="${lidar_pos_r} ${lidar_pos_p} 3.141592"/>
+        <origin xyz="${lidar_pos_x} ${lidar_pos_y} ${lidar_pos_z}" rpy="${lidar_pos_r} ${lidar_pos_p} ${lidar_pos_w}"/>
     </joint>
     <joint name="wheel_right_joint" type="continuous">
